Commit message: Gazebo_launch added with few changes in the rest

File: gdgu_robot/resource/robot_body.xacro (robot description, xacro)
@@ -23,5 +23,5 @@
     <link name="chassis_link">
         <visual>
-            <origin xyz="0.145 0.0 0.002" rpy="0.0 0.0 0.0"/>
+            <origin xyz="0.145 0.0 0.044" rpy="0.0 0.0 0.0"/>
             <geometry>
                 <box size="0.35 0.29 0.002"/>
@@ -30,5 +30,5 @@
         </visual>
         <collision>
-            <origin xyz="0.145 0.0 0.002" rpy="0.0 0.0 0.0"/>
+            <origin xyz="0.145 0.0 0.044" rpy="0.0 0.0 0.0"/>
             <geometry>
                 <box size="0.35 0.29 0.002"/>
@@ -43,5 +43,5 @@
         <parent link="base_link"/>
         <child link="lfw_link"/>
-        <origin xyz = "0.0 0.145 0.0" rpy = "-$(eval pi/2) 0.0 0.0" />
+        <origin xyz = "0.0 0.145 0.05" rpy = "-$(eval pi/2) 0.0 0.0" />
         <axis xyz="0.0 0.0 1.0"/>
     </joint>
@@ -67,5 +67,5 @@
         <parent link="base_link"/>
         <child link="rfw_link"/>
-        <origin xyz = "0.0 -0.145 0.0" rpy = "$(eval pi/2) 0.0 0.0" />
+        <origin xyz = "0.0 -0.145 0.05" rpy = "$(eval pi/2) 0.0 0.0" />
         <axis xyz="0.0 0.0 -1.0"/>
     </joint>
@@ -92,5 +92,5 @@
         <parent link="base_link"/>
         <child link="cwl1_link"/>
-        <origin xyz = "0.16 0.115 -0.04" rpy = "0 0 0"/>
+        <origin xyz = "0.16 0.115 0.01" rpy = "0 0 0"/>
         <axis xyz="1.0 1.0 1.0"/>
     </joint>
@@ -114,5 +114,5 @@
         <parent link="base_link"/>
         <child link="cwl2_link"/>
-        <origin xyz = "0.16 -0.115 -0.04" rpy = "0 0 0"/>
+        <origin xyz = "0.16 -0.115 0.01" rpy = "0 0 0"/>
         <axis xyz="1.0 1.0 1.0"/>
     </joint>
@@ -136,5 +136,5 @@
         <parent link="base_link"/>
         <child link="cwl3_link"/>
-        <origin xyz = "-0.1 0.115 -0.04" rpy = "0 0 0"/>
+        <origin xyz = "-0.1 0.115 0.01" rpy = "0 0 0"/>
         <axis xyz="1.0 1.0 1.0"/>
     </joint>
@@ -158,5 +158,5 @@
         <parent link="base_link"/>
         <child link="cwl4_link"/>
-        <origin xyz = "-0.1 -0.115 -0.04" rpy = "0 0 0"/>
+        <origin xyz = "-0.1 -0.115 0.01" rpy = "0 0 0"/>
         <axis xyz="1.0 1.0 1.0"/>
     </joint>
@@ -181,5 +181,5 @@
         <parent link="chassis_link"/>
         <child link="connector_cw1_link"/>
-        <origin xyz="0.26 0.115 -0.02" rpy="0 0 0"/>
+        <origin xyz="0.26 0.115 0.022" rpy="0 0 0"/>
     </joint>
     <link name="connector_cw1_link">
@@ -203,5 +203,5 @@
         <parent link="chassis_link"/>
         <child link="connector_cw2_link"/>
-        <origin xyz="0.26 -0.115 -0.02" rpy="0 0 0"/>
+        <origin xyz="0.26 -0.115 0.022" rpy="0 0 0"/>
     </joint>
     <link name="connector_cw2_link">
@@ -225,5 +225,5 @@
         <parent link="chassis_link"/>
         <child link="connector_cw3_link"/>
-        <origin xyz="-0.0 0.115 -0.02" rpy="0 0 0"/>
+        <origin xyz="-0.0 0.115 0.022" rpy="0 0 0"/>
     </joint>
     <link name="connector_cw3_link">
@@ -247,5 +247,5 @@
         <parent link="chassis_link"/>
         <child link="connector_cw4_link"/>
-        <origin xyz="-0.0 -0.115 -0.02" rpy="0 0 0"/>
+        <origin xyz="-0.0 -0.115 0.022" rpy="0 0 0"/>
     </joint>
     <link name="connector_cw4_link">
