Commit message: xacro update according to fortress

File: gdgu_robot/resource/gdgu_robot.urdf.xacro (robot description, xacro)
@@ -2,3 +2,4 @@
 <robot xmlns:xacro="http://www.ros.org/wiki/xacro" name = "gdgu_robot">
     <xacro:include filename="robot_body.xacro"/>
+    <xacro:include filename="gazebo_control.xacro"/>
 </robot>

File: gdgu_robot/resource/robot_body.xacro (robot description, xacro)
@@ -1,97 +1,125 @@
 <?xml version="1.0"?>
-<robot xmlns:xacro="http://www.ros.org/wiki/xacro">
+<robot xmlns:xacro="http://www.ros.org/wiki/xacro" name = "gdgu_robot">
     <xacro:include filename="robot_inertia.xacro"/>
+    <xacro:property name="chassis_length" value="0.35"/>
+    <xacro:property name="chassis_width" value="0.29"/>
+    <xacro:property name="chassis_height" value="0.002"/>
+    <xacro:property name="chassis_mass" value="2.0"/>
+    <xacro:property name="wheel_radius" value="0.05"/>
+    <xacro:property name="wheel_thickness" value="0.02"/>
+    <xacro:property name="wheel_mass" value="0.5"/>
+    <xacro:property name="wheel_offset_x" value="0.175"/>
+    <xacro:property name="wheel_offset_y" value="0.145"/>
+    <xacro:property name="wheel_offset_z" value="0.01"/>
     <material name="white">
-        <color rgba = "1 1 1 1" />
-    </material>
-     <material name="grey">
-        <color rgba = "0.25 0.25 0.25 1" />
-    </material>
-     <material name="red">
-        <color rgba = "1 0 0 1" />
-    </material>
-    <!--base link-->
+        <color rgba="1 1 1 1" />
+    </material>
+    <material name="orange">
+        <color rgba="1 0.3 0.1 1"/>
+    </material>
+    <material name="blue">
+        <color rgba="0.2 0.2 1 1"/>
+    </material>
+    <material name="black">
+        <color rgba="0 0 0 1"/>
+    </material>
+    <material name="red">
+        <color rgba="1 0 0 1"/>
+    </material>
+    <!-- BASE LINK -->
     <link name="base_link">
     </link>
-    <!-- chassis_joint -->
+    <!-- BASE_FOOTPRINT LINK -->
+    <joint name="base_footprint_joint" type="fixed">
+        <parent link="base_link"/>
+        <child link="base_footprint"/>
+        <origin xyz="0 0 0" rpy="0 0 0"/>
+    </joint>
+    <link name="base_footprint">
+    </link>
+    <!-- CHASSIS LINK -->
     <joint name="chassis_joint" type="fixed">
         <parent link="base_link"/>
         <child link="chassis_link"/>
-        <origin xyz="-0.1 0.0 0.0" rpy="0.0 0.0 0.0"/>
-    </joint>
-    <!-- chassis_link -->
+        <origin xyz="${-wheel_offset_x} 0 ${-wheel_offset_z}"/>
+    </joint>
     <link name="chassis_link">
         <visual>
-            <origin xyz="0.145 0.0 0.044" rpy="0.0 0.0 0.0"/>
-            <geometry>
-                <box size="0.35 0.29 0.002"/>
-            </geometry>
-            <material name = "white"/>
-        </visual>
-        <collision>
-            <origin xyz="0.145 0.0 0.044" rpy="0.0 0.0 0.0"/>
-            <geometry>
-                <box size="0.35 0.29 0.002"/>
-            </geometry>
-        </collision>
-        <xacro:inertial_box mass = "1" x = "0.35" y = "29" z = "0.002">
-            <origin xyz="0.145 0.0 0.002" rpy="0.0 0.0 0.0"/>
+            <origin xyz="${chassis_length/2} 0 ${chassis_height/2}"/>
+            <geometry>
+                <box size="${chassis_length} ${chassis_width} ${chassis_height}"/>
+            </geometry>
+            <material name="orange"/>
+        </visual>
+        <collision>
+            <origin xyz="${chassis_length/2} 0 ${chassis_height/2}"/>
+            <geometry>
+                <box size="${chassis_length} ${chassis_width} ${chassis_height}"/>
+            </geometry>
+        </collision>
+        <xacro:inertial_box mass="0.5" x="${chassis_length}" y="${chassis_width}" z="${chassis_height}">
+            <origin xyz="${chassis_length/2} 0 ${chassis_height/2}" rpy="0 0 0"/>
         </xacro:inertial_box>
     </link>
-    <!--wheels-->
+    <gazebo reference="chassis_link">
+        <material>Gazebo/Orange</material>
+    </gazebo>
+    <!-- LEFT WHEEL LINK -->
     <joint name="left_wheel" type="continuous">
         <parent link="base_link"/>
         <child link="lfw_link"/>
-        <origin xyz = "0.0 0.145 0.05" rpy = "-$(eval pi/2) 0.0 0.0" />
-        <axis xyz="0.0 0.0 1.0"/>
+        <origin xyz="0 ${wheel_offset_y} 0" rpy="-${pi/2} 0 0" />
+        <axis xyz="0 0 1"/>
     </joint>
     <link name="lfw_link">
         <visual>
-            <origin xyz="0.0 0.0 0.0" rpy="0.0 0.0 0.0"/>
-            <geometry>
-                <cylinder radius = "0.05" length = "0.02"/>
-            </geometry>
-            <material name = "grey"/>
-        </visual>
-        <collision>
-            <origin xyz="0.0 0.0 0.0" rpy="0.0 0.0 0.0"/>
-            <geometry>
-                <cylinder radius = "0.05" length = "0.02"/>
-            </geometry>
-        </collision>
-        <xacro:inertial_cylinder mass = "0.2" radius = "0.05" length = "0.02">
-            <origin xyz="0.0 0.0 0.0" rpy="0.0 0.0 0.0"/>
-        </xacro:inertial_cylinder>
-    </link>
+            <geometry>
+                <cylinder radius="${wheel_radius}" length="${wheel_thickness}"/>
+            </geometry>
+            <material name="blue"/>
+        </visual>
+        <collision>
+            <geometry>
+                <sphere radius="${wheel_radius}"/>
+            </geometry>
+        </collision>
+        <xacro:inertial_cylinder mass="${wheel_mass}" length="${wheel_thickness}" radius="${wheel_radius}">
+            <origin xyz="0 0 0" rpy="0 0 0"/>
+        </xacro:inertial_cylinder>
+    </link>
+    <gazebo reference="lfw_link">
+        <material>Gazebo/Blue</material>
+    </gazebo>
+    <!-- RIGHT WHEEL LINK -->
     <joint name="right_wheel" type="continuous">
         <parent link="base_link"/>
         <child link="rfw_link"/>
-        <origin xyz = "0.0 -0.145 0.05" rpy = "$(eval pi/2) 0.0 0.0" />
-        <axis xyz="0.0 0.0 -1.0"/>
+        <origin xyz="0 ${-wheel_offset_y} 0" rpy="${pi/2} 0 0" />
+        <axis xyz="0 0 -1"/>
     </joint>
     <link name="rfw_link">
         <visual>
-            <origin xyz="0.0 0.0 0.0" rpy="0.0 0.0 0.0"/>
-            <geometry>
-                <cylinder radius = "0.05" length = "0.02"/>
-            </geometry>
-            <material name = "grey"/>
-        </visual>
-        <collision>
-            <origin xyz="0.0 0.0 0.0" rpy="0.0 0.0 0.0"/>
-            <geometry>
-                <cylinder radius = "0.05" length = "0.02"/>
-            </geometry>
-        </collision>
-        <xacro:inertial_cylinder mass = "0.2" radius = "0.05" length = "0.02">
-            <origin xyz="0.0 0.0 0.0" rpy="0.0 0.0 0.0"/>
-        </xacro:inertial_cylinder>
-    </link>
+            <geometry>
+                <cylinder radius="${wheel_radius}" length="${wheel_thickness}"/>
+            </geometry>
+            <material name="blue"/>
+        </visual>
+        <collision>
+            <geometry>
+                <sphere radius="${wheel_radius}"/>
+            </geometry>
+        </collision>
+        <xacro:inertial_cylinder mass="${wheel_mass}" length="${wheel_thickness}" radius="${wheel_radius}">
+            <origin xyz="0 0 0" rpy="0 0 0"/>
+        </xacro:inertial_cylinder>
+    </link>
+    <gazebo reference="rfw_link">
+        <material>Gazebo/Blue</material>
+    </gazebo>
     <!--castor wheels-->
-    <joint name="castor_wheel1" type="continuous">
+    <joint name="castor_wheel1" type="fixed">
         <parent link="base_link"/>
         <child link="cwl1_link"/>
-        <origin xyz = "0.16 0.115 0.01" rpy = "0 0 0"/>
-        <axis xyz="1.0 1.0 1.0"/>
+        <origin xyz = "0.16 0.115 0.0" rpy = "0 0 0"/>
     </joint>
     <link name="cwl1_link">
@@ -111,9 +139,12 @@
         </xacro:inertial_sphere>
     </link>
-    <joint name="castor_wheel2" type="continuous">
+    <gazebo reference= "cwl1_link">
+        <mu1 value="0.0001"/>
+        <mu2 value="0.0001"/>
+    </gazebo>
+    <joint name="castor_wheel2" type="fixed">
         <parent link="base_link"/>
         <child link="cwl2_link"/>
         <origin xyz = "0.16 -0.115 0.01" rpy = "0 0 0"/>
-        <axis xyz="1.0 1.0 1.0"/>
     </joint>
     <link name="cwl2_link">
@@ -133,9 +164,12 @@
         </xacro:inertial_sphere>
     </link>
-    <joint name="castor_wheel3" type="continuous">
+    <gazebo reference= "cwl2_link">
+        <mu1 value="0.0001"/>
+        <mu2 value="0.0001"/>
+    </gazebo>
+    <joint name="castor_wheel3" type="fixed">
         <parent link="base_link"/>
         <child link="cwl3_link"/>
         <origin xyz = "-0.1 0.115 0.01" rpy = "0 0 0"/>
-        <axis xyz="1.0 1.0 1.0"/>
     </joint>
     <link name="cwl3_link">
@@ -155,9 +189,12 @@
         </xacro:inertial_sphere>
     </link>
-    <joint name="castor_wheel4" type="continuous">
+    <gazebo reference= "cwl3_link">
+        <mu1 value="0.0001"/>
+        <mu2 value="0.0001"/>
+    </gazebo>
+    <joint name="castor_wheel4" type="fixed">
         <parent link="base_link"/>
         <child link="cwl4_link"/>
         <origin xyz = "-0.1 -0.115 0.01" rpy = "0 0 0"/>
-        <axis xyz="1.0 1.0 1.0"/>
     </joint>
     <link name="cwl4_link">
@@ -177,4 +214,8 @@
         </xacro:inertial_sphere>
     </link>
+    <gazebo reference= "cwl4_link">
+        <mu1 value="0.0001"/>
+        <mu2 value="0.0001"/>
+    </gazebo>
     <!--connectors for castor wheels-->
     <joint name="connector_cw1_joint" type="fixed">
@@ -188,5 +229,5 @@
                 <cylinder radius="0.005" length="0.04"/>
             </geometry>
-            <material name="grey"/>
+            <material name="black"/>
         </visual>
         <collision>
@@ -210,5 +251,5 @@
                 <cylinder radius="0.005" length="0.04"/>
             </geometry>
-            <material name="grey"/>
+            <material name="black"/>
         </visual>
         <collision>
@@ -232,5 +273,5 @@
                 <cylinder radius="0.005" length="0.04"/>
             </geometry>
-            <material name="grey"/>
+            <material name="black"/>
         </visual>
         <collision>
@@ -254,5 +295,5 @@
                 <cylinder radius="0.005" length="0.04"/>
             </geometry>
-            <material name="grey"/>
+            <material name="black"/>
         </visual>
         <collision>
