Commit message: Changes

File: gdgu_robot/resource/gazebo_control.xacro (robot description, xacro)
@@ -2,5 +2,5 @@
 <robot xmlns:xacro="http://www.ros.org/wiki/xacro" name = "gdgu_robot">
     <gazebo>
-        <plugin name= "ignition::gazebo::systems::DiffDrive" filename = "libignition-gazebo-diff-drive-system.so">
+        <plugin name="ignition::gazebo::systems::DiffDrive" filename="libignition-gazebo-diff-drive-system.so">
             <!--Wheel Info-->
             <left_joint>left_wheel</left_joint>
@@ -24,5 +24,5 @@
             <min_angular_velocity>-1</min_angular_velocity>
         </plugin>
-        <plugin name= "ignition::gazebo::systems::JointStatePublisher" filename= "libignition-gazebo-joint-state-publisher-system.so">
+        <plugin name="ignition::gazebo::systems::JointStatePublisher" filename="libignition-gazebo-joint-state-publisher-system.so">
             <topic>joint_states</topic>
             <joint_name>left_wheel</joint_name>

File: gdgu_robot/resource/robot_body.xacro (robot description, xacro)
@@ -10,6 +10,10 @@
     <xacro:property name="wheel_mass" value="0.5"/>
     <xacro:property name="wheel_offset_x" value="0.175"/>
-    <xacro:property name="wheel_offset_y" value="0.145"/>
+    <xacro:property name="wheel_offset_y" value="0.155"/>
     <xacro:property name="wheel_offset_z" value="0.01"/>
+    <xacro:property name="caster_wheel_radius" value="0.01"/>
+    <xacro:property name="caster_wheel_mass" value="0.01"/>
+    <xacro:property name="caster_wheel_offset_x" value="0.015"/>
+    <xacro:property name="caster_wheel_offset_z" value="${wheel_offset_z - wheel_radius + caster_wheel_radius}"/>
     <material name="white">
         <color rgba="1 1 1 1" />
@@ -114,118 +118,121 @@
         </xacro:inertial_cylinder>
     </link>
-    <gazebo reference="rfw_link">
+    <gazebo reference="rfw_wheel">
         <material>Gazebo/Blue</material>
     </gazebo>
     <!--castor wheels-->
-    <joint name="castor_wheel1" type="fixed">
-        <parent link="base_link"/>
-        <child link="cwl1_link"/>
-        <origin xyz = "0.16 0.115 0.0" rpy = "0 0 0"/>
-    </joint>
-    <link name="cwl1_link">
-        <visual>
-            <geometry>
-                <sphere radius = "0.01"/>
-            </geometry>
-            <material name="red"/>
-        </visual>
-        <collision>
-            <geometry>
-                <sphere radius = "0.01"/>
-            </geometry>
-        </collision>
-        <xacro:inertial_sphere mass = "0.1" radius = "0.01">
-            <origin xyz="0.0 0.0 0.0" rpy="0.0 0.0 0.0"/>
+    <joint name="caster_wheel1_joint" type="fixed">
+        <parent link="chassis_link"/>
+        <child link="caster_wheel1_link"/>
+        <origin xyz="${caster_wheel_offset_x} 0.125 ${caster_wheel_offset_z}"/>
+    </joint>
+    <link name="caster_wheel1_link">
+        <visual>
+            <geometry>
+                <sphere radius="${caster_wheel_radius}"/>
+            </geometry>
+            <material name="white"/>
+        </visual>
+        <collision>
+            <geometry>
+                <sphere radius="${caster_wheel_radius}"/>
+            </geometry>
+        </collision>
+        <xacro:inertial_sphere mass="${caster_wheel_mass}" radius="${caster_wheel_radius}">
+            <origin xyz="0 0 0" rpy="0 0 0"/>
         </xacro:inertial_sphere>
     </link>
-    <gazebo reference= "cwl1_link">
-        <mu1 value="0.0001"/>
-        <mu2 value="0.0001"/>
-    </gazebo>
-    <joint name="castor_wheel2" type="fixed">
-        <parent link="base_link"/>
-        <child link="cwl2_link"/>
-        <origin xyz = "0.16 -0.115 0.01" rpy = "0 0 0"/>
-    </joint>
-    <link name="cwl2_link">
-        <visual>
-            <geometry>
-                <sphere radius = "0.01"/>
-            </geometry>
-            <material name="red"/>
-        </visual>
-        <collision>
-            <geometry>
-                <sphere radius = "0.01"/>
-            </geometry>
-        </collision>
-        <xacro:inertial_sphere mass = "0.1" radius = "0.01">
-            <origin xyz="0.0 0.0 0.0" rpy="0.0 0.0 0.0"/>
+    <gazebo reference="caster_wheel1_link">
+        <material>Gazebo/Red</material>
+        <mu1 value="0.001"/>
+        <mu2 value="0.001"/>
+    </gazebo>
+    <joint name="caster_wheel2_joint" type="fixed">
+        <parent link="chassis_link"/>
+        <child link="caster_wheel2_link"/>
+        <origin xyz="${caster_wheel_offset_x} -0.125 ${caster_wheel_offset_z}"/>
+    </joint>
+    <link name="caster_wheel2_link">
+        <visual>
+            <geometry>
+                <sphere radius="${caster_wheel_radius}"/>
+            </geometry>
+            <material name="white"/>
+        </visual>
+        <collision>
+            <geometry>
+                <sphere radius="${caster_wheel_radius}"/>
+            </geometry>
+        </collision>
+        <xacro:inertial_sphere mass="${caster_wheel_mass}" radius="${caster_wheel_radius}">
+            <origin xyz="0 0 0" rpy="0 0 0"/>
         </xacro:inertial_sphere>
     </link>
-    <gazebo reference= "cwl2_link">
-        <mu1 value="0.0001"/>
-        <mu2 value="0.0001"/>
-    </gazebo>
-    <joint name="castor_wheel3" type="fixed">
-        <parent link="base_link"/>
-        <child link="cwl3_link"/>
-        <origin xyz = "-0.1 0.115 0.01" rpy = "0 0 0"/>
-    </joint>
-    <link name="cwl3_link">
-        <visual>
-            <geometry>
-                <sphere radius = "0.01"/>
-            </geometry>
-            <material name="red"/>
-        </visual>
-        <collision>
-            <geometry>
-                <sphere radius = "0.01"/>
-            </geometry>
-        </collision>
-        <xacro:inertial_sphere mass = "0.1" radius = "0.01">
-            <origin xyz="0.0 0.0 0.0" rpy="0.0 0.0 0.0"/>
+    <gazebo reference="caster_wheel2_link">
+        <material>Gazebo/Red</material>
+        <mu1 value="0.001"/>
+        <mu2 value="0.001"/>
+    </gazebo>
+<joint name="caster_wheel3_joint" type="fixed">
+        <parent link="chassis_link"/>
+        <child link="caster_wheel3_link"/>
+        <origin xyz="${caster_wheel_offset_x + 0.29} 0.125 ${caster_wheel_offset_z}"/>
+    </joint>
+    <link name="caster_wheel3_link">
+        <visual>
+            <geometry>
+                <sphere radius="${caster_wheel_radius}"/>
+            </geometry>
+            <material name="white"/>
+        </visual>
+        <collision>
+            <geometry>
+                <sphere radius="${caster_wheel_radius}"/>
+            </geometry>
+        </collision>
+        <xacro:inertial_sphere mass="${caster_wheel_mass}" radius="${caster_wheel_radius}">
+            <origin xyz="0 0 0" rpy="0 0 0"/>
         </xacro:inertial_sphere>
     </link>
-    <gazebo reference= "cwl3_link">
-        <mu1 value="0.0001"/>
-        <mu2 value="0.0001"/>
-    </gazebo>
-    <joint name="castor_wheel4" type="fixed">
-        <parent link="base_link"/>
-        <child link="cwl4_link"/>
-        <origin xyz = "-0.1 -0.115 0.01" rpy = "0 0 0"/>
-    </joint>
-    <link name="cwl4_link">
-        <visual>
-            <geometry>
-                <sphere radius = "0.01"/>
-            </geometry>
-            <material name="red"/>
-        </visual>
-        <collision>
-            <geometry>
-                <sphere radius = "0.01"/>
-            </geometry>
-        </collision>
-        <xacro:inertial_sphere mass = "0.1" radius = "0.01">
-            <origin xyz="0.0 0.0 0.0" rpy="0.0 0.0 0.0"/>
+    <gazebo reference="caster_wheel3_link">
+        <material>Gazebo/Red</material>
+        <mu1 value="0.001"/>
+        <mu2 value="0.001"/>
+    </gazebo>
+<joint name="caster_wheel4_joint" type="fixed">
+        <parent link="chassis_link"/>
+        <child link="caster_wheel4_link"/>
+        <origin xyz="${caster_wheel_offset_x + 0.29} -0.125 ${caster_wheel_offset_z}"/>
+    </joint>
+    <link name="caster_wheel4_link">
+        <visual>
+            <geometry>
+                <sphere radius="${caster_wheel_radius}"/>
+            </geometry>
+            <material name="white"/>
+        </visual>
+        <collision>
+            <geometry>
+                <sphere radius="${caster_wheel_radius}"/>
+            </geometry>
+        </collision>
+        <xacro:inertial_sphere mass="${caster_wheel_mass}" radius="${caster_wheel_radius}">
+            <origin xyz="0 0 0" rpy="0 0 0"/>
         </xacro:inertial_sphere>
     </link>
-    <gazebo reference= "cwl4_link">
-        <mu1 value="0.0001"/>
-        <mu2 value="0.0001"/>
-    </gazebo>
-    <!--connectors for castor wheels-->
+    <gazebo reference="caster_wheel4_link">
+        <material>Gazebo/Red</material>
+        <mu1 value="0.001"/>
+        <mu2 value="0.001"/>
+    </gazebo>
     <joint name="connector_cw1_joint" type="fixed">
-        <parent link="chassis_link"/>
+        <parent link="caster_wheel1_link"/>
         <child link="connector_cw1_link"/>
-        <origin xyz="0.26 0.115 0.022" rpy="0 0 0"/>
+        <origin xyz="0.0 0.0 0.02" rpy="0 0 0"/>
     </joint>
     <link name="connector_cw1_link">
         <visual>
             <geometry>
-                <cylinder radius="0.005" length="0.04"/>
+                <cylinder radius="0.005" length="0.022"/>
             </geometry>
             <material name="black"/>
@@ -233,8 +240,8 @@
         <collision>
             <geometry>
-                <cylinder radius="0.005" length="0.04"/>
-            </geometry>
-        </collision>
-        <xacro:inertial_cylinder mass = "0.1" radius = "0.005" length = "0.04">
+                <cylinder radius="0.005" length="0.022"/>
+            </geometry>
+        </collision>
+        <xacro:inertial_cylinder mass = "0.1" radius = "0.005" length = "0.022">
             <origin xyz="0.0 0.0 0.0" rpy="0.0 0.0 0.0"/>
         </xacro:inertial_cylinder>
@@ -242,12 +249,12 @@
     <!-- Connector for castor wheel 2 -->
     <joint name="connector_cw2_joint" type="fixed">
-        <parent link="chassis_link"/>
+        <parent link="caster_wheel2_link"/>
         <child link="connector_cw2_link"/>
-        <origin xyz="0.26 -0.115 0.022" rpy="0 0 0"/>
+        <origin xyz="0.0 0.0 0.02" rpy="0 0 0"/>
     </joint>
     <link name="connector_cw2_link">
         <visual>
             <geometry>
-                <cylinder radius="0.005" length="0.04"/>
+                <cylinder radius="0.005" length="0.022"/>
             </geometry>
             <material name="black"/>
@@ -255,8 +262,8 @@
         <collision>
             <geometry>
-                <cylinder radius="0.005" length="0.04"/>
-            </geometry>
-        </collision>
-        <xacro:inertial_cylinder mass = "0.1" radius = "0.005" length = "0.04">
+                <cylinder radius="0.005" length="0.022"/>
+            </geometry>
+        </collision>
+        <xacro:inertial_cylinder mass = "0.1" radius = "0.005" length = "0.022">
             <origin xyz="0.0 0.0 0.0" rpy="0.0 0.0 0.0"/>
         </xacro:inertial_cylinder>
@@ -264,12 +271,12 @@
     <!-- Connector for castor wheel 3 -->
     <joint name="connector_cw3_joint" type="fixed">
-        <parent link="chassis_link"/>
+        <parent link="caster_wheel3_link"/>
         <child link="connector_cw3_link"/>
-        <origin xyz="-0.0 0.115 0.022" rpy="0 0 0"/>
+        <origin xyz="0.0 0.0 0.02" rpy="0 0 0"/>
     </joint>
     <link name="connector_cw3_link">
         <visual>
             <geometry>
-                <cylinder radius="0.005" length="0.04"/>
+                <cylinder radius="0.005" length="0.022"/>
             </geometry>
             <material name="black"/>
@@ -277,8 +284,8 @@
         <collision>
             <geometry>
-                <cylinder radius="0.005" length="0.04"/>
-            </geometry>
-        </collision>
-        <xacro:inertial_cylinder mass = "0.1" radius = "0.005" length = "0.04">
+                <cylinder radius="0.005" length="0.022"/>
+            </geometry>
+        </collision>
+        <xacro:inertial_cylinder mass = "0.1" radius = "0.005" length = "0.022">
             <origin xyz="0.0 0.0 0.0" rpy="0.0 0.0 0.0"/>
         </xacro:inertial_cylinder>
@@ -286,12 +293,12 @@
     <!-- Connector for castor wheel 4 -->
     <joint name="connector_cw4_joint" type="fixed">
-        <parent link="chassis_link"/>
+        <parent link="caster_wheel4_link"/>
         <child link="connector_cw4_link"/>
-        <origin xyz="-0.0 -0.115 0.022" rpy="0 0 0"/>
+        <origin xyz="0.0 0.0 0.02" rpy="0 0 0"/>
     </joint>
     <link name="connector_cw4_link">
         <visual>
             <geometry>
-                <cylinder radius="0.005" length="0.04"/>
+                <cylinder radius="0.005" length="0.022"/>
             </geometry>
             <material name="black"/>
@@ -299,8 +306,8 @@
         <collision>
             <geometry>
-                <cylinder radius="0.005" length="0.04"/>
-            </geometry>
-        </collision>
-        <xacro:inertial_cylinder mass = "0.1" radius = "0.005" length = "0.04">
+                <cylinder radius="0.005" length="0.022"/>
+            </geometry>
+        </collision>
+        <xacro:inertial_cylinder mass = "0.1" radius = "0.005" length = "0.022">
             <origin xyz="0.0 0.0 0.0" rpy="0.0 0.0 0.0"/>
         </xacro:inertial_cylinder>

Commit message: final_changes_for_keyboard_control

File: gdgu_robot/resource/gazebo_control.xacro (robot description, xacro)
@@ -2,5 +2,5 @@
 <robot xmlns:xacro="http://www.ros.org/wiki/xacro" name = "gdgu_robot">
     <gazebo>
-        <plugin name="ignition::gazebo::systems::DiffDrive" filename="libignition-gazebo-diff-drive-system.so">
+        <plugin filename="gz-sim-diff-drive-system" name="gz::sim::systems::DiffDrive">
             <!--Wheel Info-->
             <left_joint>left_wheel</left_joint>
@@ -9,20 +9,12 @@
             <wheel_radius>0.05</wheel_radius>
             <!--input-->
-            <odom_publish_frequency>10</odom_publish_frequency>
+            <odom_publish_frequency>100</odom_publish_frequency>
             <topic>cmd_vel</topic>
             <!--output "what needs to be shown in the output"-->
             <odom_topic>odom</odom_topic>
-            <tf_topic>tf</tf_topic>
-            <frame_id>odom</frame_id>
-            <child_frame_id>base_link</child_frame_id>
             <!--limits "set according to the motor requirements"-->
             <max_linear_accelaration>1</max_linear_accelaration>
-            <max_angular_acceleration>1</max_angular_acceleration>
-            <max_linear_velocity>1</max_linear_velocity>
-            <min_linear_velocity>-1</min_linear_velocity>
-            <max_angular_velocity>1</max_angular_velocity>
-            <min_angular_velocity>-1</min_angular_velocity>
         </plugin>
-        <plugin name="ignition::gazebo::systems::JointStatePublisher" filename="libignition-gazebo-joint-state-publisher-system.so">
+        <plugin filename="gz-sim-joint-state-publisher-system" name="gz::sim::systems::JointStatePublisher">
             <topic>joint_states</topic>
             <joint_name>left_wheel</joint_name>

File: gdgu_robot/resource/robot.xacro (robot description, xacro)
@@ -1,5 +1,31 @@
 <?xml version="1.0"?>
 <robot xmlns:xacro="http://www.ros.org/wiki/xacro" name = "gdgu_robot">
-    <xacro:include filename="robot_inertia.xacro"/>
+    <xacro:macro name="inertial_box" params="mass x y z *origin">
+        <inertial>
+            <xacro:insert_block name="origin"/>
+            <mass value="${mass}"/>
+            <inertia ixx="${(1/12) * mass * (y*y+z*z)}" ixy="0.0" ixz="0.0"
+                    iyy="${(1/12) * mass * (x*x+z*z)}" iyz="0.0"
+                    izz="${(1/12) * mass * (x*x+y*y)}" />
+        </inertial>
+    </xacro:macro>
+    <xacro:macro name="inertial_sphere" params="mass radius *origin">
+        <inertial>
+            <xacro:insert_block name="origin"/>
+            <mass value="${mass}"/>
+            <inertia ixx="${(2/5) * mass * (radius*radius)}" ixy="0.0" ixz="0.0"
+                    iyy="${(2/5) * mass * (radius*radius)}" iyz="0.0"
+                    izz="${(2/5) * mass * (radius*radius)}" />
+        </inertial>
+    </xacro:macro>
+    <xacro:macro name="inertial_cylinder" params="mass radius length *origin">
+        <inertial>
+            <xacro:insert_block name="origin"/>
+            <mass value="${mass}"/>
+            <inertia ixx="${(1/12) * mass * (3*radius*radius + length*length)}" ixy="0.0" ixz="0.0"
+                    iyy="${(1/12) * mass * (3*radius*radius + length*length)}" iyz="0.0"
+                    izz="${(1/2) * mass * (radius*radius)}" />
+        </inertial>
+    </xacro:macro>
     <xacro:property name="chassis_length" value="0.35"/>
     <xacro:property name="chassis_width" value="0.29"/>
@@ -62,5 +88,5 @@
             </geometry>
         </collision>
-        <xacro:inertial_box mass="0.5" x="${chassis_length}" y="${chassis_width}" z="${chassis_height}">
+        <xacro:inertial_box mass="${chassis_mass}" x="${chassis_length}" y="${chassis_width}" z="${chassis_height}">
             <origin xyz="${chassis_length/2} 0 ${chassis_height/2}" rpy="0 0 0"/>
         </xacro:inertial_box>
@@ -313,3 +339,24 @@
         </xacro:inertial_cylinder>
     </link>
+    <gazebo>
+        <plugin filename="gz-sim-diff-drive-system" name="gz::sim::systems::DiffDrive">
+            <!--Wheel Info-->
+            <left_joint>left_wheel</left_joint>
+            <right_joint>right_wheel</right_joint>
+            <wheel_separation>0.31</wheel_separation>
+            <wheel_radius>0.05</wheel_radius>
+            <!--input-->
+            <odom_publish_frequency>100</odom_publish_frequency>
+            <topic>cmd_vel</topic>
+            <!--output "what needs to be shown in the output"-->
+            <odom_topic>odom</odom_topic>
+            <!--limits "set according to the motor requirements"-->
+            <max_linear_acceleration>1</max_linear_acceleration>
+        </plugin>
+        <plugin filename="gz-sim-joint-state-publisher-system" name="gz::sim::systems::JointStatePublisher">
+            <topic>joint_states</topic>
+            <joint_name>left_wheel</joint_name>
+            <joint_name>right_wheel</joint_name>
+        </plugin>
+    </gazebo>
 </robot>

Commit message: adding ultrasonic sensor

File: gdgu_robot/resource/gazebo_control.xacro (robot description, xacro)
@@ -13,4 +13,6 @@
             <!--output "what needs to be shown in the output"-->
             <odom_topic>odom</odom_topic>
+            <frame_id>odom</frame_id>
+            <child_frame_id>base_link</child_frame_id>
             <!--limits "set according to the motor requirements"-->
             <max_linear_accelaration>1</max_linear_accelaration>
@@ -20,5 +22,10 @@
             <joint_name>left_wheel</joint_name>
             <joint_name>right_wheel</joint_name>
+            <joint_name>rotor_joint</joint_name>
         </plugin>
+       <!-- <plugin filename="gz-sim-joint-state-publisher-system" name="gz::sim::systems::JointStatePublisher">
+            <topic>stepper_joint_states</topic>
+            <joint_name>rotor_joint</joint_name>
+        </plugin> -->
     </gazebo>
 </robot>

File: gdgu_robot/resource/gdgu_robot.urdf.xacro (robot description, xacro)
@@ -3,3 +3,4 @@
     <xacro:include filename="robot_body.xacro"/>
     <xacro:include filename="gazebo_control.xacro"/>
+    <xacro:include filename="ultrasonic.xacro"/>
 </robot>

File: gdgu_robot/resource/robot.urdf (robot description, URDF)
Before this commit: robot gdgu_robot, 13 links, 12 joints
Links:
- added link ray_link
- added link rotor_link, mass 0.01; collision cylinder length=0.01 radius=.005; visual cylinder length=0.01 radius=.005
- added link stepper_link, mass 0.1; collision box size=0.02 0.01 0.02; visual box size=0.02 0.02 0.01
- added link ultrasonic_link, mass 0.1; collision box size=0.045 0.02 0.015; visual mesh filename=package://gdgu_robot/meshes/ULTRASONIC_INFRARED.STL scale=0.001 0.0004 0.0009
- link chassis_link: mass 2.0 -> 0.5
Joints:
- added joint ray_joint: type fixed, parent ultrasonic_link, child ray_link, origin xyz=0.0 0.15 0.05 rpy=0.0 0.0 0.0
- added joint rotor_joint: type revolute, parent stepper_link, child rotor_link, origin xyz=0.0 0.0 0.01 rpy=0.0 0.0 0.0, axis 0 0 1, limit lower=-0.6545 upper=0.6545 effort=1 velocity=0.5
- added joint stepper_joint: type fixed, parent chassis_link, child stepper_link, origin xyz=0.34 0.0 0.01 rpy=0.0 0.0 0.0
- added joint ultrasonic_joint: type fixed, parent rotor_link, child ultrasonic_link, origin xyz=0.0 -0.02 0.0 rpy=1.57 0 1.57

File: gdgu_robot/resource/robot_inertia.xacro (robot description, xacro)
@@ -29,3 +29,21 @@
         </inertial>
     </xacro:macro>
+  <!-- Conversion macros -->
+    <xacro:property name="cm2m"    value="${1/100.0}"/>
+    <xacro:property name="mm2m"    value="${1/1000.0}"/>
+    <xacro:property name="in2m"    value="0.0254"/>
+    <xacro:property name="deg2rad" value="${pi/180.0}"/>
+  <!-- Material colors -->
+    <material name="material_black">
+        <color rgba="0.1 0.1 0.1 1"/>
+    </material>
+    <material name="material_darkgray">
+        <color rgba="0.3 0.3 0.3 1"/>
+    </material>
+    <material name="sensor_blue">
+        <color rgba="0.1 0.2 0.8 1"/>
+    </material>
+    <material name="material_lightgray">
+        <color rgba="0.5 0.5 0.5 1"/>
+    </material>
 </robot>
