Commit message: changes to world file

File: gdgu_robot/resource/gdgu_hardware.xacro (robot description, xacro)
@@ -76,4 +76,13 @@
         <axis xyz="0 0 1"/>
     </joint>
+    <transmission name="left_wheel_trans" type="SimpleTransmission">
+    <type>transmission_interface/SimpleTransmission</type>
+    <actuator name="left_wheel_motor">
+      <mechanicalReduction>1</mechanicalReduction>
+    </actuator>
+    <joint name="left_wheel">
+      <hardwareInterface>VelocityJointInterface</hardwareInterface>
+    </joint>
+    </transmission>
     <link name="lfw_link">
         <visual>
@@ -102,4 +111,13 @@
         <axis xyz="0 0 -1"/>
     </joint>
+    <transmission name="right_wheel_trans" type="SimpleTransmission">
+    <type>transmission_interface/SimpleTransmission</type>
+    <actuator name="right_wheel_motor">
+      <mechanicalReduction>1</mechanicalReduction>
+    </actuator>
+    <joint name="right_wheel">
+      <hardwareInterface>VelocityJointInterface</hardwareInterface>
+    </joint>
+    </transmission>
     <link name="rfw_link">
         <visual>

File: gdgu_robot/resource/robot_hardware.urdf (robot description, URDF)
Before this commit: robot gdgu_robot, 18 links, 17 joints
Links:
- removed link cam_support_link
- removed link camera_link
- removed link rotor_link
- removed link stepper_link
- removed link ultrasonic_link
Joints:
- removed joint camera_joint
- removed joint camera_supp_joint
- removed joint rotor_joint
- removed joint stepper_joint
- removed joint ultrasonic_joint

File: gdgu_robot/resource/robot_hardware.urdf.xacro (robot description, xacro)
@@ -1,7 +1,5 @@
 <?xml version="1.0"?>
 <robot xmlns:xacro="http://www.ros.org/wiki/xacro" name = "gdgu_robot">
-    <xacro:include filename="robot_body.xacro"/>
+    <xacro:include filename="gdgu_hardware.xacro"/>
     <xacro:include filename="gazebo_control.xacro"/>
-    <xacro:include filename="ultrasonic.xacro"/>
-    <xacro:include filename="camera.xacro"/>
 </robot>

File: gdgu_robot/resource/ultrasonic.xacro (robot description, xacro)
@@ -21,9 +21,9 @@
         </collision>
         <xacro:inertial_box mass="0.1" x="0.02" y="0.02" z="0.01">
-        <origin xyz="0.34 0.0 0.01" rpy="0.0 0.0 0.0"/>
+            <origin xyz="0.34 0.0 0.01" rpy="0.0 0.0 0.0"/>
         </xacro:inertial_box>
     </link>
      <gazebo reference="stepper_link">
-        <material>Gazebo/Green</material>
+        <material>Gazebo/Black</material>
     </gazebo>
     <joint name="rotor_joint" type="revolute">
@@ -76,18 +76,10 @@
         </inertial>
     </link>
-    <!--joint and link for ray direction-->
-    <joint name="ray_joint" type="fixed">
-        <parent link="ultrasonic_link"/>
-        <child link="ray_link"/>
-        <origin xyz="0.0 0.15 0.05" rpy="0.0 0.0 0.0"/>
-    </joint>
-    <link name="ray_link">
-    </link>
-    <gazebo reference="ray_link">
-        <sensor name="ultrasonic" type="ray">
+    <gazebo reference="ultrasonic_link">
+        <sensor name="ultrasonic" type="gpu_lidar">
+            <pose> 0 -0.02 0 -1.57 0 1.57 </pose>
             <update_rate>5</update_rate>
             <always_on>1</always_on>
             <visualize>1</visualize>
-            <topic>ultrasonic_sensor</topic>
             <ray>
                 <scan>
@@ -95,11 +87,11 @@
                         <samples>1</samples>
                         <resolution>1</resolution>
-                        <min_angle>0</min_angle>
-                        <max_angle>15</max_angle>
+                        <min_angle>-0.309</min_angle>
+                        <max_angle>0.309</max_angle>
                     </horizontal>
                 </scan>
                 <range>
                     <min>0.03</min>
-                    <max>0.4</max>
+                    <max>4.0</max>
                     <resolution>0.02</resolution>
                 </range>
@@ -110,4 +102,6 @@
                 </noise>
             </ray>
+            <topic>scan</topic>
+            <gz_frame_id>ultrasonic_link</gz_frame_id>
         </sensor>
     </gazebo>
